File: quadripod_board/quadripod_v2.brd (EAGLE design)
At the start: 50 x 83 mm, 21 parts

Commit message: update board, some checks to come
Parts:
- removed 5V_RASPI: M02PTH, 7robot:1X02
- added U$1: M03X2T, 7robot:2X03
Connections:
- net N$12 renamed RX
- net N$13 renamed TX
- new net N$17: PCB1.J1.14, U$1.2
- new net N$18: PCB1.J2.3, U$1.6
- new net N$19: PCB1.J2.15, U$1.5
- new net N$20: PCB1.J1.15, U$1.4
- net 5V_NANO: now also U$1.3; no longer 5V_RASPI.2
- net GND: now also U$1.1; no longer 5V_RASPI.1
Routing:
- net N$20: track 0.00 -> 110.8 mm, vias 0 -> 1
- net N$17: track 0.00 -> 107.4 mm, vias 0 -> 1
- net N$18: track 0.00 -> 33.2 mm, vias 0 -> 1
- net N$19: track 0.00 -> 9.37 mm, vias 0 -> 1
- net 5V_NANO: track 42.9 -> 46.1 mm, vias 0 -> 1
