File: quadripod_board/quadripod_v2.sch (EAGLE design)
At the start: 21 parts

Commit message: update board, some checks to come
Parts:
- removed 5V_RASPI: M02PTH, 7robot:M02PTH
- added U$1: M03X2T, 7robot:M03X2T
Connections:
- net N$12 renamed RX
- net N$13 renamed TX
- new net N$17: PCB1.D11/MOSI, U$1.2
- new net N$18: PCB1.RST.2, U$1.6
- new net N$19: PCB1.D13/SCK, U$1.5
- new net N$20: PCB1.D12/MISO, U$1.4
- net 5V_NANO: now also U$1.3; no longer 5V_RASPI.2
- net GND: now also U$1.1; no longer 5V_RASPI.1
Changed lines of the file:
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@@
 <part name="BA_CON" library="7robot" deviceset="M02" device="PTH" value="M02PTH"/>
 <part name="UART_CON" library="7robot" deviceset="M02" device="PTH" value="M02PTH"/>
-<part name="5V_RASPI" library="7robot" deviceset="M02" device="PTH" value="M02PTH"/>
 <part name="PI1" library="7robot" deviceset="STCMS_2" device=""/>
 <part name="PI2" library="7robot" deviceset="STCMS_2" device=""/>
 <part name="PI3" library="7robot" deviceset="STCMS_2" device=""/>
+<part name="U$1" library="7robot" deviceset="M03X2" device="T"/>
 </parts>
 <sheets>
@@
 <attribute name="NAME" x="-22.86" y="31.242" size="1.778" layer="95"/>
 </instance>
-<instance part="5V_RASPI" gate="G$1" x="76.2" y="-15.24" smashed="yes" rot="R90">
-<attribute name="VALUE" x="81.28" y="-17.78" size="1.778" layer="96" rot="R90"/>
-<attribute name="NAME" x="70.358" y="-17.78" size="1.778" layer="95" rot="R90"/>
-</instance>
 <instance part="PI1" gate="G$1" x="58.42" y="139.7" smashed="yes" rot="R90">
 <attribute name="NAME" x="62.2301" y="136.8425" size="1.778" layer="95" rot="R180"/>
@@
 <instance part="PI3" gate="G$1" x="58.42" y="83.82" smashed="yes" rot="R90">
 <attribute name="NAME" x="62.2301" y="80.9625" size="1.778" layer="95" rot="R180"/>
+</instance>
+<instance part="U$1" gate="G$1" x="68.58" y="-17.78" smashed="yes" rot="R270">
+<attribute name="VALUE" x="60.96" y="-15.24" size="1.778" layer="96" rot="R270"/>
+<attribute name="NAME" x="74.422" y="-15.24" size="1.778" layer="95" rot="R270"/>
 </instance>
 </instances>
@@
 </segment>
 <segment>
-<wire x1="88.9" y1="-7.62" x2="88.9" y2="0" width="0.1524" layer="91"/>
 <pinref part="GND7" gate="1" pin="GND"/>
-<pinref part="5V_RASPI" gate="G$1" pin="1"/>
-<wire x1="76.2" y1="-7.62" x2="88.9" y2="-7.62" width="0.1524" layer="91"/>
+<pinref part="U$1" gate="G$1" pin="1"/>
+<wire x1="66.04" y1="-25.4" x2="66.04" y2="-35.56" width="0.1524" layer="91"/>
+<wire x1="66.04" y1="-35.56" x2="88.9" y2="-35.56" width="0.1524" layer="91"/>
+<wire x1="88.9" y1="-35.56" x2="88.9" y2="0" width="0.1524" layer="91"/>
 </segment>
 <segment>
@@
 <segment>
 <pinref part="PCB1" gate="G$1" pin="5V"/>
-<wire x1="48.26" y1="20.32" x2="66.04" y2="20.32" width="0.1524" layer="91"/>
-<wire x1="66.04" y1="20.32" x2="66.04" y2="-7.62" width="0.1524" layer="91"/>
-<pinref part="5V_RASPI" gate="G$1" pin="2"/>
-<wire x1="66.04" y1="-7.62" x2="73.66" y2="-7.62" width="0.1524" layer="91"/>
+<wire x1="48.26" y1="20.32" x2="60.96" y2="20.32" width="0.1524" layer="91"/>
 <label x="68.58" y="12.7" size="1.778" layer="95"/>
+<pinref part="U$1" gate="G$1" pin="3"/>
+<wire x1="60.96" y1="20.32" x2="66.04" y2="20.32" width="0.1524" layer="91"/>
+<wire x1="71.12" y1="-25.4" x2="83.82" y2="-25.4" width="0.1524" layer="91"/>
+<wire x1="83.82" y1="-25.4" x2="83.82" y2="20.32" width="0.1524" layer="91"/>
+<wire x1="83.82" y1="20.32" x2="66.04" y2="20.32" width="0.1524" layer="91"/>
 </segment>
 <segment>
@@
 </segment>
 </net>
-<net name="N$12" class="0">
+<net name="RX" class="0">
 <segment>
 <pinref part="PCB1" gate="G$1" pin="D0/RX"/>
 <pinref part="UART_CON" gate="G$1" pin="1"/>
 <wire x1="-12.7" y1="25.4" x2="10.16" y2="25.4" width="0.1524" layer="91"/>
-</segment>
-</net>
-<net name="N$13" class="0">
+<label x="0" y="22.86" size="1.778" layer="95"/>
+</segment>
+</net>
+<net name="TX" class="0">
 <segment>
 <pinref part="PCB1" gate="G$1" pin="D1/TX"/>
 <pinref part="UART_CON" gate="G$1" pin="2"/>
 <wire x1="-12.7" y1="27.94" x2="10.16" y2="27.94" width="0.1524" layer="91"/>
+<label x="0" y="30.48" size="1.778" layer="95"/>
 </segment>
 </net>
@@
 </segment>
 </net>
+<net name="N$19" class="0">
+<segment>
+<pinref part="PCB1" gate="G$1" pin="D13/SCK"/>
+<pinref part="U$1" gate="G$1" pin="5"/>
+<wire x1="48.26" y1="-7.62" x2="68.58" y2="-7.62" width="0.1524" layer="91"/>
+<wire x1="68.58" y1="-7.62" x2="68.58" y2="-10.16" width="0.1524" layer="91"/>
+</segment>
+</net>
+<net name="N$20" class="0">
+<segment>
+<pinref part="U$1" gate="G$1" pin="4"/>
+<wire x1="71.12" y1="-10.16" x2="71.12" y2="-2.54" width="0.1524" layer="91"/>
+<wire x1="71.12" y1="-2.54" x2="60.96" y2="-2.54" width="0.1524" layer="91"/>
+<wire x1="60.96" y1="-2.54" x2="60.96" y2="-35.56" width="0.1524" layer="91"/>
+<wire x1="60.96" y1="-35.56" x2="7.62" y2="-35.56" width="0.1524" layer="91"/>
+<pinref part="PCB1" gate="G$1" pin="D12/MISO"/>
+<wire x1="7.62" y1="-35.56" x2="7.62" y2="-7.62" width="0.1524" layer="91"/>
+<wire x1="7.62" y1="-7.62" x2="10.16" y2="-7.62" width="0.1524" layer="91"/>
+</segment>
+</net>
+<net name="N$17" class="0">
+<segment>
+<pinref part="U$1" gate="G$1" pin="2"/>
+<wire x1="68.58" y1="-25.4" x2="68.58" y2="-38.1" width="0.1524" layer="91"/>
+<wire x1="68.58" y1="-38.1" x2="5.08" y2="-38.1" width="0.1524" layer="91"/>
+<wire x1="5.08" y1="-38.1" x2="5.08" y2="-5.08" width="0.1524" layer="91"/>
+<pinref part="PCB1" gate="G$1" pin="D11/MOSI"/>
+<wire x1="5.08" y1="-5.08" x2="10.16" y2="-5.08" width="0.1524" layer="91"/>
+</segment>
+</net>
+<net name="N$18" class="0">
+<segment>
+<pinref part="U$1" gate="G$1" pin="6"/>
+<pinref part="PCB1" gate="G$1" pin="RST.2"/>
+<wire x1="66.04" y1="-10.16" x2="66.04" y2="22.86" width="0.1524" layer="91"/>
+<wire x1="66.04" y1="22.86" x2="48.26" y2="22.86" width="0.1524" layer="91"/>
+</segment>
+</net>
