File: quadripod_board/quadripod_v3Rc.brd (EAGLE design)
At the start: 48 x 85 mm, 19 parts

Commit message: upate of the board
Parts:
- removed BA_CON: M02PTH, SparkFun-Connectors:1X02_LONGPADS
- added BAT: M02PTH, SparkFun-Connectors:1X02_LONGPADS
- renumbered I2C_CON to I2C, S_C1 to C1, S_C2 to C2, S_C3 to C3, S_C4 to C4, S_E1 to E1, S_E2 to E2, S_E3 to E3, S_E4 to E4, UART_CON to UART
Connections:
- net +12V: now also BAT.2; no longer BA_CON.2
- net GND: now also BAT.1; no longer BA_CON.1
Routing:
- net GND: track 40.0 -> 143.4 mm
- net 5VB: track 13.5 -> 92.0 mm
- net 5V_RPI: track 0.00 -> 67.2 mm
- net SC4: track 0.00 -> 44.6 mm, vias 0 -> 2
- net SE4: track 0.00 -> 40.0 mm, vias 0 -> 2
- net SC3: track 0.00 -> 35.4 mm, vias 0 -> 2
- net SE3: track 0.00 -> 32.1 mm, vias 0 -> 2
- net SC2: track 0.00 -> 30.7 mm, vias 0 -> 2
- net SE1: track 0.00 -> 28.5 mm, vias 0 -> 2
- net SC1: track 0.00 -> 23.8 mm, vias 0 -> 2
- net SE2: track 0.00 -> 19.2 mm, vias 0 -> 2
- net 3V3: track 0.00 -> 11.8 mm
- net I2C_VCC: track 0.00 -> 3.57 mm
- net I2C_SDA: track 0.00 -> 3.52 mm
- net I2C_SCL: track 0.00 -> 3.52 mm
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Other:
- board text added: "3.3v"
- board text added: "5v"
- board text added: "Rx"
- board text added: "SCL"
- board text added: "SDA"
- board text added: "Thib-s v3.0 Rev C"
- board text added: "Tx"
- board text added: "Vin"
- board text added: "gnd"
- board text removed: "Thib-s v3.0 Rev B"
