File: quadripod_board/quadripod_v3Rc.sch (EAGLE design)
At the start: 19 parts

Commit message: upate of the board
Parts:
- renumbered BA_CON to BAT, I2C_CON to I2C, S_C1 to C1, S_C2 to C2, S_C3 to C3, S_C4 to C4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
